File: hardware/dsbi-digital-part.kicad_pcb (KiCad board)
At the start: 2 copper layers, 34 x 51.3 mm, 4 parts

Commit message: Improvements
Changed lines of the file:
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@@
       (dashed_line_gap_ratio 3.000000)
       (svgprecision 4)
-      (plotframeref true)
+      (plotframeref false)
       (viasonmask false)
       (mode 1)
@@
         (effects (font (size 1 1) (thickness 0.15)))
     )
-    (fp_text value "ESP32-WROOM" (at 1.484902 -4.067388 180) (layer "F.Fab")
+    (fp_text value "ESP32-WROOM" (at 1.484902 -4.067388 180) (layer "F.SilkS")
         (effects (font (size 1 1) (thickness 0.15)))
     )
@@
   (gr_rect (start 12.206902 12.442612) (end 46.242902 63.750612)
     (stroke (width 0.1) (type default)) (fill none) (layer "Edge.Cuts"))
-  (gr_text "Damn\nSimple\nBrainwave\nInterface\n(Digital processor)\nrev 1.0" (at 36.082902 48.510612) (layer "B.Cu")
-    (effects (font (size 0.8 0.8) (thickness 0.2) bold) (justify left bottom mirror))
-  )
   (gr_text "IN+" (at 36.082902 50.288612 270) (layer "F.SilkS")
     (effects (font (size 1 1) (thickness 0.1)) (justify left bottom))
@@
     (effects (font (size 1 1) (thickness 0.1)) (justify left bottom))
   )
+  (gr_text "Damn\nSimple\nBrainwave\nInterface\n(Digital processor)\nrev 1.0" (at 25.4 45.72) (layer "F.SilkS")
+    (effects (font (size 0.8 0.8) (thickness 0.2) bold) (justify left bottom))
+  )
   (gr_text "TX" (at 33.57101 14.460557) (layer "F.SilkS")
